File: hydrabus-shield-template.sch (KiCad schematic (older format))
At the start: 4 parts, among them J1 CONN_02X07, J2 CONN_02X10, J3 CONN_02X10, J4 CONN_01X06

Commit message: pcb/sch: updated footprints
Parts:
- J1: footprint Pin_Headers:Pin_Header_Straight_2x07 -> umetronics:Hydrabus_Shield_Conn_2x07
- J2, J3: footprint Pin_Headers:Pin_Header_Straight_2x10 -> umetronics:Hydrabus_Shield_Conn_2x10
- J4: footprint Pin_Headers:Pin_Header_Straight_1x06 -> umetronics:Hydrabus_Shield_Conn_1x06
Changed lines of the file:
@@
 F 0 "J3" H 1450 5750 50  0000 C CNN
 F 1 "CONN_02X10" V 1450 5200 50  0000 C CNN
-F 2 "Pin_Headers:Pin_Header_Straight_2x10" H 1450 4000 50  0001 C CNN
+F 2 "umetronics:Hydrabus_Shield_Conn_2x10" H 1450 4000 50  0001 C CNN
 F 3 "" H 1450 4000 50  0000 C CNN
 	1    1450 5200
@@
 F 0 "J2" H 1450 3850 50  0000 C CNN
 F 1 "CONN_02X10" V 1450 3300 50  0000 C CNN
-F 2 "Pin_Headers:Pin_Header_Straight_2x10" H 1450 2100 50  0001 C CNN
+F 2 "umetronics:Hydrabus_Shield_Conn_2x10" H 1450 2100 50  0001 C CNN
 F 3 "" H 1450 2100 50  0000 C CNN
 	1    1450 3300
@@
 F 0 "J1" H 1450 1850 50  0000 C CNN
 F 1 "CONN_02X07" V 1450 1450 50  0000 C CNN
-F 2 "Pin_Headers:Pin_Header_Straight_2x07" H 1450 250 50  0001 C CNN
+F 2 "umetronics:Hydrabus_Shield_Conn_2x07" H 1450 250 50  0001 C CNN
 F 3 "" H 1450 250 50  0000 C CNN
 	1    1450 1450
@@
 F 0 "J4" H 1800 7450 50  0000 C CNN
 F 1 "CONN_01X06" V 1900 7100 50  0000 C CNN
-F 2 "Pin_Headers:Pin_Header_Straight_1x06" H 1800 7100 50  0001 C CNN
+F 2 "umetronics:Hydrabus_Shield_Conn_1x06" H 1800 7100 50  0001 C CNN
 F 3 "" H 1800 7100 50  0000 C CNN
 	1    1800 7100
